Commit message: lib is not loaded

File: orbita2d_description/ros2_control/orbita2d.ros2_control.xacro (robot description, xacro)
@@ -7,5 +7,5 @@
         <!-- Use real hardware. -->
         <xacro:unless value="$(arg use_fake_hardware)">
-          <plugin>orbita2d_system_hwi/Orbita2dSerialSystem</plugin>
+          <plugin>orbita2d_system_hwi/Orbita2dSystem</plugin>
           <param name="config_file">${config_file}</param>
         </xacro:unless>

File: orbita2d_description/urdf/orbita2d.urdf.xacro (robot description, xacro)
@@ -4,8 +4,8 @@
   <xacro:include filename="$(find orbita2d_description)/ros2_control/orbita2d.ros2_control.xacro"/>
     <material name="orbita2dmetal">
-        <color rgba="0.85 0.85 0.85 1"/>
+        <color rgba="0.85 0.85 0.85 1.0"/>
     </material>
     <material name="orbita2dgrey">
-        <color rgba="0.8 0.8 0.8 1"/>
+        <color rgba="0.8 0.8 0.8 1.0"/>
     </material>
   <xacro:macro name="joint2axis" params="joint">

File: orbita2d_description/urdf/test_orbita2d.urdf.xacro (robot description, xacro)
@@ -1,5 +1,5 @@
 <?xml version="1.0" ?>
 <robot xmlns:xacro="http://www.ros.org/wiki/xacro" name="test_orbita2d">
-  <xacro:arg name="use_fake_hardware" default="true"/>
+  <xacro:arg name="use_fake_hardware" default="false"/>
   <xacro:arg name="use_gazebo" default="false"/>
   <xacro:include filename="$(find orbita2d_description)/urdf/inertial_primitives.urdf.xacro"/>
@@ -8,5 +8,5 @@
   <xacro:arg name="config_file" default="$(find orbita2d_description)/config/fake.yaml"/>
   <!-- MODEL PARAMETERS -->
-  <xacro:property name="base_collision" value="false"/>
+  <xacro:property name="base_collision" value="true"/>
   <xacro:property name="base_visual" value="true"/>
   <xacro:property name="damping" value="0.1"/>
@@ -22,5 +22,5 @@
   <!-- MODEL PARAMETERS -->
     <material name="torsoblack">
-        <color rgba="0.5 0.5 0.5 1"/>
+        <color rgba="0.5 0.5 0.5 1.0"/>
     </material>
   <link name="world"/>
@@ -71,7 +71,14 @@
     config_file="$(arg config_file)"
   />
-  <link name="tip"/>
+  <link name="tip">
+    <visual>
+      <origin xyz="0 0 0" rpy="0 0.0 0"/>
+      <geometry>
+          <sphere radius="0.05"/>
+      </geometry>
+    </visual>
+  </link>
   <joint name="tip_joint" type="fixed">
-    <origin xyz="0 0 -0.2" rpy="0 0 0"/>
+    <origin xyz="0 0 -0.3" rpy="0 0 0"/>
     <parent link="shoulder_ball_link"/>
     <child link="tip"/>

Commit message: test launch seems ok

File: orbita2d_description/ros2_control/orbita2d.ros2_control.xacro (robot description, xacro)
@@ -2,5 +2,5 @@
 <robot xmlns:xacro="http://www.ros.org/wiki/xacro">
   <xacro:include filename="$(find orbita2d_description)/ros2_control/joint.ros2_control.xacro"/>
-  <xacro:macro name="orbita2d_control" params="name joint1 joint2 config_file">
+  <xacro:macro name="orbita2d_control" params="name joint1 joint2 config_file axis1_inverted axis2_inverted">
     <ros2_control name="${name}" type="system">
       <hardware>
@@ -9,4 +9,6 @@
           <plugin>orbita2d_system_hwi/Orbita2dSystem</plugin>
           <param name="config_file">${config_file}</param>
+          <param name="axis1_inverted">${axis1_inverted}</param>
+          <param name="axis2_inverted">${axis2_inverted}</param>
         </xacro:unless>
         <xacro:if value="$(arg use_fake_hardware)">

File: orbita2d_description/urdf/orbita2d.urdf.xacro (robot description, xacro)
@@ -20,5 +20,5 @@
     </xacro:if>
   </xacro:macro>
-  <xacro:macro name="orbita2d" params="name parent length radius mass xyz rpy damping friction joint1 joint2 joint1_min_angle joint1_max_angle joint2_min_angle joint2_max_angle config_file">
+  <xacro:macro name="orbita2d" params="name parent length radius mass xyz rpy damping friction joint1 joint2 joint1_min_angle joint1_max_angle joint2_min_angle joint2_max_angle config_file axis1_inverted axis2_inverted">
     <!--
       Orbita 2 dof
@@ -96,4 +96,5 @@
       joint1="${joint1}" joint2="${joint2}"
       config_file="${config_file}"
+      axis1_inverted="${axis1_inverted}" axis2_inverted="${axis2_inverted}"
     />
   </xacro:macro>

File: orbita2d_description/urdf/test_orbita2d.urdf.xacro (robot description, xacro)
@@ -70,4 +70,5 @@
     joint2_min_angle="-${pi/2}" joint2_max_angle="0.0"
     config_file="$(arg config_file)"
+    axis1_inverted="0" axis2_inverted="1"
   />
   <link name="tip">

Commit message: Remove axes inversion from ROS.

File: orbita2d_description/ros2_control/orbita2d.ros2_control.xacro (robot description, xacro)
@@ -2,5 +2,5 @@
 <robot xmlns:xacro="http://www.ros.org/wiki/xacro">
   <xacro:include filename="$(find orbita2d_description)/ros2_control/joint.ros2_control.xacro"/>
-  <xacro:macro name="orbita2d_control" params="name joint1 joint2 config_file axis1_inverted axis2_inverted">
+  <xacro:macro name="orbita2d_control" params="name joint1 joint2 config_file ">
     <ros2_control name="${name}" type="system">
       <hardware>
@@ -9,6 +9,4 @@
           <plugin>orbita2d_system_hwi/Orbita2dSystem</plugin>
           <param name="config_file">${config_file}</param>
-          <param name="axis1_inverted">${axis1_inverted}</param>
-          <param name="axis2_inverted">${axis2_inverted}</param>
         </xacro:unless>
         <xacro:if value="$(arg use_fake_hardware)">

File: orbita2d_description/urdf/orbita2d.urdf.xacro (robot description, xacro)
@@ -20,5 +20,5 @@
     </xacro:if>
   </xacro:macro>
-  <xacro:macro name="orbita2d" params="name parent length radius mass xyz rpy damping friction joint1 joint2 joint1_min_angle joint1_max_angle joint2_min_angle joint2_max_angle config_file axis1_inverted axis2_inverted">
+  <xacro:macro name="orbita2d" params="name parent length radius mass xyz rpy damping friction joint1 joint2 joint1_min_angle joint1_max_angle joint2_min_angle joint2_max_angle config_file">
     <!--
       Orbita 2 dof
@@ -96,5 +96,4 @@
       joint1="${joint1}" joint2="${joint2}"
       config_file="${config_file}"
-      axis1_inverted="${axis1_inverted}" axis2_inverted="${axis2_inverted}"
     />
   </xacro:macro>

File: orbita2d_description/urdf/test_orbita2d.urdf.xacro (robot description, xacro)
@@ -70,5 +70,4 @@
     joint2_min_angle="-${pi/2}" joint2_max_angle="0.0"
     config_file="$(arg config_file)"
-    axis1_inverted="0" axis2_inverted="1"
   />
   <link name="tip">
