Commit message: small change in urdf for colors

File: orbita2d_description/urdf/orbita2d.urdf.xacro (robot description, xacro)
@@ -2,11 +2,12 @@
 <robot xmlns:xacro="http://www.ros.org/wiki/xacro">
   <xacro:include filename="$(find pollen_generic_description)/urdf/inertial_primitives.urdf.xacro"/>
+  <xacro:include filename="$(find pollen_generic_description)/urdf/materials.urdf.xacro"/>
   <xacro:include filename="$(find orbita2d_description)/ros2_control/orbita2d.ros2_control.xacro"/>
-    <material name="orbita2dmetal">
-        <color rgba="0.85 0.85 0.85 1.0"/>
-    </material>
-    <material name="orbita2dgrey">
-        <color rgba="0.8 0.8 0.8 1.0"/>
-    </material>
+    <!-- <material name="orbita2dmetal"> -->
+    <!--     <color rgba="0.85 0.85 0.85 1.0"/> -->
+    <!-- </material> -->
+    <!-- <material name="orbita2dgrey"> -->
+    <!--     <color rgba="0.8 0.8 0.8 1.0"/> -->
+    <!-- </material> -->
   <xacro:macro name="joint2axis" params="joint">
     <xacro:if value="${joint == 'roll'}">
@@ -55,5 +56,6 @@
 	  <box size="${radius*2.5} ${radius*2.0} ${length}"/>
       	</geometry>
-      	<material name= "orbita2dmetal"/>
+      	<!-- <material name= "orbita2dmetal"/> -->
+	<xacro:orbita2dmetal/>
       </visual>
       <xacro:inertial_cuboid mass="${mass*0.49}" xyz="0 0 ${-length/2}"  rpy="0 0 0" x_length="${radius*2}" y_length="${radius*2}" z_length="${length}"/>
@@ -77,5 +79,6 @@
           <sphere radius="${radius*1.2}"/>
       	</geometry>
-      	<material name="orbita2dgrey"/>
+      	<!-- <material name="orbita2dgrey"/> -->
+	<xacro:orbita2dgrey/>
       </visual>
       <collision>

Commit message: mesh

File: orbita2d_description/urdf/orbita2d.urdf.xacro (robot description, xacro)
@@ -15,8 +15,8 @@
     </xacro:if>
     <xacro:if value="${joint == 'pitch'}">
-      <axis xyz="0 1 0"/>
+      <axis xyz="0 0 1"/>
     </xacro:if>
     <xacro:if value="${joint == 'yaw'}">
-      <axis xyz="0 0 1"/>
+      <axis xyz="0 1 0"/>
     </xacro:if>
   </xacro:macro>
@@ -26,15 +26,46 @@
     link                      (joint)
     ${parent}                 (${name}_joint1)
-      ${name}_dummy_link      (${name}_joint2)
+      ${name}_first_link      (${name}_joint2)
         ${name}_link          (${name}_ball_joint)
           ${name}_ball_link
     -->
-    <link name="${name}_dummy_link">
-      <xacro:inertial_cuboid mass="${mass*0.01}" xyz="0 0 0"  rpy="0 0 0" x_length="${radius*2}" y_length="${radius*2}" z_length="${length}"/>
+    <!-- used to "place" the joint with the correct axis. For some reason rotation of the inertia patrix does not work... -->
+    <link name="${name}_dummy_link1">
     </link>
-    <joint name="${name}_${joint1}" type="revolute">
+    <joint name="${name}_dummy_1" type="fixed">
       <origin xyz="${xyz}" rpy="${rpy}"/>
       <parent link="${parent}"/>
-      <child link="${name}_dummy_link"/>
+      <child link="${name}_dummy_link1"/>
+    </joint>
+    <link name="${name}_dummy_link2">
+    </link>
+    <joint name="${name}_dummy_2" type="fixed">
+      <origin xyz="0 0 0" rpy="1.5707963267948966 0 0"/>
+      <parent link="${name}_dummy_link1"/>
+      <child link="${name}_dummy_link2"/>
+    </joint>
+    <link name="${name}_first_link">
+      <visual>
+      	<origin xyz="0 0 0" rpy="0 0 0"/>
+      	<geometry>
+	  <mesh filename="package://orbita2d_description/meshes/2D_sphere_visual.dae" />
+	  <!-- <mesh filename="package://orbita2d_description/meshes/Orbita2D_Link.dae" /> -->
+      	</geometry>
+      </visual>
+      <inertial>
+      	<!-- <origin xyz="0.0 0 0" rpy="1.5707963267948966 0 0"/> -->  <!-- rotation does not work? -->
+      	<origin xyz="0.000096 -0.000015 -0.01777" rpy="0 0 0"/>
+	<mass value="0.487"/>
+	 <inertia ixx="0.000577881945" ixy="-8.085000000000001e-7" ixz="-6.962790000000001e-7"
+		  iyx="-8.085000000000001e-7" iyy="0.000573075516" iyz="2.44386e-7"
+		  izx="-6.962790000000001e-7" izy="2.44386e-7" izz="0.000243343676"/>
+      </inertial>
+    </link>
+    <!-- First joint  -->
+    <joint name="${name}_${joint1}" type="revolute">
+      <origin xyz="0 0 0" rpy="0 0 0"/>
+      <!-- <parent link="${parent}"/> -->
+      <parent link="${name}_dummy_link2"/>
+      <child link="${name}_first_link"/>
       <xacro:joint2axis joint="${joint1}"/>
       <limit lower="${joint1_min_angle}" upper="${joint1_max_angle}" effort="1000.0" velocity="100.0"/>
@@ -42,56 +73,23 @@
       <dynamics damping="${damping}" friction="${friction}"/>
     </joint>
-    <link name="${name}_link">
-      <collision>
-      	<origin xyz="0 0 ${-length/2}" rpy="0 0 0"/>
-      	<geometry>
-          <!-- <cylinder length="${length}" radius="${radius}"/> -->
-	  <box size="${radius*2.5} ${radius*2.0} ${length}"/>
-      	</geometry>
-      </collision>
-      <visual>
-      	<origin xyz="0 0 ${-length/2}" rpy="0 0 0"/>
-      	<geometry>
-          <!-- <cylinder length="${length}" radius="${radius}"/> -->
-	  <box size="${radius*2.5} ${radius*2.0} ${length}"/>
-      	</geometry>
-      	<!-- <material name= "orbita2dmetal"/> -->
-	<xacro:orbita2dmetal/>
-      </visual>
-      <xacro:inertial_cuboid mass="${mass*0.49}" xyz="0 0 ${-length/2}"  rpy="0 0 0" x_length="${radius*2}" y_length="${radius*2}" z_length="${length}"/>
+    <!-- Used to get back to the correct orientation -->
+    <link name="${name}_dummy_link3">
+    </link>
+    <joint name="${name}_dummy_3" type="fixed">
+      <origin xyz="0 0 0" rpy="-1.5707963267948966 0 0"/>
+      <parent link="${name}_first_link"/>
+      <child link="${name}_dummy_link3"/>
+    </joint>
+    <!-- Output link -->
+    <link name="${name}_ball_link">
     </link>
     <joint name="${name}_${joint2}" type="revolute">
-      <origin xyz="0 0 0" rpy="0 0 0"/>
-      <parent link="${name}_dummy_link"/>
-      <child link="${name}_link"/>
+      <origin xyz="0 0 0" rpy=" 0 0 0"/>
+      <parent link="${name}_dummy_link3"/>
+      <child link="${name}_ball_link"/>
       <xacro:joint2axis joint="${joint2}"/>
       <limit lower="${joint2_min_angle}" upper="${joint2_max_angle}" effort="1000.0" velocity="100.0"/>
       <safety_controller k_velocity="500" k_position="500" soft_lower_limit="-3.1415" soft_upper_limit="3.1415" />
       <dynamics damping="${damping}" friction="${friction}"/>
-    </joint>
-    <gazebo reference="${name}_link">
-      <material>Gazebo/Orange</material>
-    </gazebo>
-    <link name="${name}_ball_link">
-      <visual>
-      	<origin xyz="0 0 0" rpy="0 0 0"/>
-      	<geometry>
-          <sphere radius="${radius*1.2}"/>
-      	</geometry>
-      	<!-- <material name="orbita2dgrey"/> -->
-	<xacro:orbita2dgrey/>
-      </visual>
-      <collision>
-      	<origin xyz="0 0 0" rpy="0 0 0"/>
-      	<geometry>
-          <sphere radius="${radius*1.2}"/>
-      	</geometry>
-      </collision>
-      <xacro:inertial_sphere mass="${mass*0.5}" diameter="${2*radius*1.2}"/>
-    </link>
-    <joint name="${name}_ball_joint" type="fixed">
-      <origin xyz="0 0 0" rpy="0 0 0"/>
-      <parent link="${name}_link"/>
-      <child link="${name}_ball_link"/>
     </joint>
     <xacro:orbita2d_control

File: orbita2d_description/urdf/test_orbita2d.urdf.xacro (robot description, xacro)
@@ -18,5 +18,5 @@
   <xacro:property name="arm_offset_y" value="-0.1913"/>
   <xacro:property name="arm_offset_z" value="0.025"/>
-  <xacro:property name="arm_offset_yaw" value="0.2617993877991494"/>
+  <xacro:property name="arm_offset_yaw" value="0.2617993877991494"/> <!-- 15 degrees -->
   <xacro:property name="reflect" value="1"/>
   <!-- MODEL PARAMETERS -->

Commit message: wip

File: orbita2d_description/urdf/orbita2d.urdf.xacro (robot description, xacro)
@@ -3,11 +3,4 @@
   <xacro:include filename="$(find pollen_generic_description)/urdf/inertial_primitives.urdf.xacro"/>
   <xacro:include filename="$(find pollen_generic_description)/urdf/materials.urdf.xacro"/>
-  <xacro:include filename="$(find orbita2d_description)/ros2_control/orbita2d.ros2_control.xacro"/>
-    <!-- <material name="orbita2dmetal"> -->
-    <!--     <color rgba="0.85 0.85 0.85 1.0"/> -->
-    <!-- </material> -->
-    <!-- <material name="orbita2dgrey"> -->
-    <!--     <color rgba="0.8 0.8 0.8 1.0"/> -->
-    <!-- </material> -->
   <xacro:macro name="joint2axis" params="joint">
     <xacro:if value="${joint == 'roll'}">
@@ -15,8 +8,8 @@
     </xacro:if>
     <xacro:if value="${joint == 'pitch'}">
-      <axis xyz="0 0 1"/>
+      <axis xyz="0 1 0"/>
     </xacro:if>
     <xacro:if value="${joint == 'yaw'}">
-      <axis xyz="0 1 0"/>
+      <axis xyz="0 0 1"/>
     </xacro:if>
   </xacro:macro>
@@ -24,12 +17,19 @@
     <!--
       Orbita 2 dof
-    link                      (joint)
-    ${parent}                 (${name}_joint1)
-      ${name}_first_link      (${name}_joint2)
-        ${name}_link          (${name}_ball_joint)
-          ${name}_ball_link
+    link                         (joint)
+    ${parent}                    (${name}_dummy_1) fixed
+      ${name}_dummy_link1        (${name}_dummy_2) fixed
+        ${name}_dummy_link2      (${name}_joint1) revolute
+          ${name}_first_link     (${name}_joint2) revolute
+      	    ${name}_ball_link    (${name}_dummy_out) fixed
+	      ${name}_fix_link
     -->
-    <!-- used to "place" the joint with the correct axis. For some reason rotation of the inertia patrix does not work... -->
+    <!-- used to "place" the joint with the correct axis. For some reason rotation of the inertia matrix does not work... -->
     <link name="${name}_dummy_link1">
+      <inertial>
+        <origin xyz="0.0 0.0 0.0" rpy="0.0 0.0 0.0"/>
+        <mass value="0.001"/>
+        <inertia ixx="1.0e-6" ixy="1.0e-8" ixz="1.0e-8" iyy="1.0e-6" iyz="1.0e-8" izz="1.0e-6"/>
+      </inertial>
     </link>
     <joint name="${name}_dummy_1" type="fixed">
@@ -39,7 +39,25 @@
     </joint>
     <link name="${name}_dummy_link2">
+      <inertial>
+        <origin xyz="0.0 0.0 0.0" rpy="0.0 0.0 0.0"/>
+        <mass value="0.001"/>
+        <inertia ixx="1.0e-6" ixy="1.0e-8" ixz="1.0e-8" iyy="1.0e-6" iyz="1.0e-8" izz="1.0e-6"/>
+      </inertial>
     </link>
+    <!-- used to rotatate the joint to respect the conventional axis -->
     <joint name="${name}_dummy_2" type="fixed">
+    <xacro:if value="${name == 'r_shoulder'}">
+      <origin xyz="0 0 0" rpy="-1.5707963267948966 0 0"/>
+    </xacro:if>
+    <xacro:if value="${name == 'l_shoulder'}">
       <origin xyz="0 0 0" rpy="1.5707963267948966 0 0"/>
+    </xacro:if>
+    <xacro:if value="${name == 'r_elbow'}">
+      <origin xyz="0 0 0" rpy="3.141592 0 1.5707963267948966"/>
+    </xacro:if>
+    <xacro:if value="${name == 'l_elbow'}">
+      <origin xyz="0 0 0" rpy="3.141592 0 -1.5707963267948966"/>
+    </xacro:if>
+      <!-- <origin xyz="0 0 0" rpy="0 0 0"/> -->
       <parent link="${name}_dummy_link1"/>
       <child link="${name}_dummy_link2"/>
@@ -47,10 +65,27 @@
     <link name="${name}_first_link">
       <visual>
-      	<origin xyz="0 0 0" rpy="0 0 0"/>
+      	<!-- <origin xyz="0 0 0" rpy="0 0 0"/> -->
+    <xacro:if value="${name == 'r_shoulder'}">
+      <origin xyz="0 0 0" rpy="1.5707963267948966 0 0"/>
+    </xacro:if>
+    <xacro:if value="${name == 'l_shoulder'}">
+      <origin xyz="0 0 0" rpy="-1.5707963267948966 0 0"/>
+    </xacro:if>
+    <xacro:if value="${name == 'r_elbow'}">
+      <origin xyz="0 0 0" rpy="3.141592 0 -1.5707963267948966"/>
+    </xacro:if>
+    <xacro:if value="${name == 'l_elbow'}">
+      <origin xyz="0 0 0" rpy="3.141592 0 1.5707963267948966"/>
+    </xacro:if>
       	<geometry>
-	  <mesh filename="package://orbita2d_description/meshes/2D_sphere_visual.dae" />
-	  <!-- <mesh filename="package://orbita2d_description/meshes/Orbita2D_Link.dae" /> -->
+	  <!-- <mesh filename="file://$(find arm_description)/meshes/Orbita2D_ball.dae" /> -->
+	  <mesh filename="file://$(find orbita2d_description)/meshes/2D_sphere_visual.dae" />
       	</geometry>
       </visual>
+	<!-- <collision> -->
+	<!--   <geometry> -->
+	<!--     <sphere radius="0.0425"/> -->
+	<!--   </geometry> -->
+	<!-- </collision> -->
       <inertial>
       	<!-- <origin xyz="0.0 0 0" rpy="1.5707963267948966 0 0"/> -->  <!-- rotation does not work? -->
@@ -68,28 +103,63 @@
       <parent link="${name}_dummy_link2"/>
       <child link="${name}_first_link"/>
+      <!-- axis1 -->
       <xacro:joint2axis joint="${joint1}"/>
+      <!-- <axis xyz="0 0 -1"/> -->
       <limit lower="${joint1_min_angle}" upper="${joint1_max_angle}" effort="1000.0" velocity="100.0"/>
+      <safety_controller k_velocity="500" k_position="500" soft_lower_limit="-3.141592" soft_upper_limit="3.1415" />
+      <dynamics damping="${damping}" friction="${friction}"/>
+    </joint>
+    <!-- <!-\- Used to get back to the correct orientation -\-> -->
+    <!-- <link name="${name}_dummy_link3"> -->
+    <!-- </link> -->
+    <!-- <joint name="${name}_dummy_3" type="fixed"> -->
+    <!--   <!-\- <origin xyz="0 0 0" rpy="-1.5707963267948966 0 0"/> -\-> -->
+    <!--   <origin xyz="0 0 0" rpy="3.141592653589793 0 0"/> -->
+    <!--   <parent link="${name}_first_link"/> -->
+    <!--   <child link="${name}_dummy_link3"/> -->
+    <!-- </joint> -->
+    <!-- Output link -->
+    <link name="${name}_ball_link">
+      <inertial>
+        <origin xyz="0.0 0.0 0.0" rpy="0.0 0.0 0.0"/>
+        <mass value="0.001"/>
+        <inertia ixx="1.0e-6" ixy="1.0e-8" ixz="1.0e-8" iyy="1.0e-6" iyz="1.0e-8" izz="1.0e-6"/>
+      </inertial>
+    </link>
+    <joint name="${name}_${joint2}" type="revolute">
+      <origin xyz="0 0 0" rpy=" 0 0 0"/>
+      <parent link="${name}_first_link"/>
+      <child link="${name}_ball_link"/>
+      <!-- axis2 -->
+      <xacro:joint2axis joint="${joint2}"/>
+      <!-- <axis xyz="1 0 0"/> -->
+      <limit lower="${joint2_min_angle}" upper="${joint2_max_angle}" effort="1000.0" velocity="100.0"/>
       <safety_controller k_velocity="500" k_position="500" soft_lower_limit="-3.1415" soft_upper_limit="3.1415" />
       <dynamics damping="${damping}" friction="${friction}"/>
     </joint>
-    <!-- Used to get back to the correct orientation -->
-    <link name="${name}_dummy_link3">
+    <link name="${name}_fix_link">
+      <inertial>
+        <origin xyz="0.0 0.0 0.0" rpy="0.0 0.0 0.0"/>
+        <mass value="0.001"/>
+        <inertia ixx="1.0e-6" ixy="1.0e-8" ixz="1.0e-8" iyy="1.0e-6" iyz="1.0e-8" izz="1.0e-6"/>
+      </inertial>
     </link>
-    <joint name="${name}_dummy_3" type="fixed">
-      <origin xyz="0 0 0" rpy="-1.5707963267948966 0 0"/>
-      <parent link="${name}_first_link"/>
-      <child link="${name}_dummy_link3"/>
-    </joint>
-    <!-- Output link -->
-    <link name="${name}_ball_link">
-    </link>
-    <joint name="${name}_${joint2}" type="revolute">
-      <origin xyz="0 0 0" rpy=" 0 0 0"/>
-      <parent link="${name}_dummy_link3"/>
-      <child link="${name}_ball_link"/>
-      <xacro:joint2axis joint="${joint2}"/>
-      <limit lower="${joint2_min_angle}" upper="${joint2_max_angle}" effort="1000.0" velocity="100.0"/>
-      <safety_controller k_velocity="500" k_position="500" soft_lower_limit="-3.1415" soft_upper_limit="3.1415" />
-      <dynamics damping="${damping}" friction="${friction}"/>
+    <!-- used to rotate the joint to respect the conventional axis -->
+    <joint name="${name}_dummy_out" type="fixed">
+    <xacro:if value="${name == 'r_shoulder'}">
+      <origin xyz="0 0 0" rpy="1.5707963267948966 0 0"/>
+    </xacro:if>
+    <xacro:if value="${name == 'l_shoulder'}">
+      <origin xyz="0 0 0" rpy="1.5707963267948966 0 0"/>
+    </xacro:if>
+    <xacro:if value="${name == 'r_elbow'}">
+      <origin xyz="0 0 0" rpy="3.141592 0 1.5707963267948966"/>
+    </xacro:if>
+    <xacro:if value="${name == 'l_elbow'}">
+      <origin xyz="0 0 0" rpy="3.141592 0 1.5707963267948966"/>
+    </xacro:if>
+      <!-- <origin xyz="0 0 0" rpy="0 0 0"/> -->
+      <parent link="${name}_ball_link"/>
+      <child link="${name}_fix_link"/>
     </joint>
     <xacro:orbita2d_control
